File: shield_servo_adc_sw_gpio_led.sch (KiCad schematic (older format))
At the start: 38 parts, among them J1 srv,adc, J10 Conn_02x01, J2 srv,adc, J3 srv,adc, J4 srv,adc, J5 srv,adc, J6 srv,adc, J7 srv,adc, J8 srv,adc, J9 usart,i2c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

Commit message: tlp627
Parts:
- removed C1, C2, C3, C4, C5, C6, C7, C8: 1u, Capacitor_SMD:C_0603_1608Metric, symbol Device:C_Small
- removed F2: 30V6A, Fuse:Fuse_Bourns_MF-RHT600, symbol Device:Polyfuse_Small
- removed J1, J2, J3, J4, J5, J6, J7, J8: srv,adc, Connector_JST:JST_PH_S3B-PH-K_1x03_P2.00mm_Horizontal, symbol Connector:Conn_01x03_Male
- removed JP1, JP10, JP11, JP12, JP13, JP14, JP15, JP16, JP2, JP3, JP4, JP5, JP6, JP7, JP8, JP9: jumper, Jumper:SolderJumper-3_P1.3mm_Open_RoundedPad1.0x1.5mm_NumberLabels, symbol Jumper:SolderJumper_3_Bridged12
- added J? (x8): Solenoid, symbol Connector:Conn_01x02_Male
- added RN?: R_Pack08, symbol Device:R_Pack08
- added U? (x8): TLP627, Package_DIP:DIP-4_W7.62mm, symbol Isolator:TLP627
Connections:
- net AD0: now also RN?.1 (R1.1)
- net AD1: now also RN?.2 (R2.1)
- net AD2: now also RN?.3 (R3.1)
- net AD3: now also RN?.4 (R4.1)
- net AD4: now also RN?.5 (R5.1)
- net AD5: now also RN?.6 (R6.1)
- net AD6: now also RN?.7 (R7.1)
- net AD7: now also RN?.8 (R8.1)
- net GND: now also U?.2, U?.2, U?.2, U?.2, U?.2, U?.2, U?.2, U?.2; no longer C9.2, J10.1 (Pin_1)
- net VCC: now also U?.4, U?.4, U?.4, U?.4, U?.4, U?.4, U?.4, U?.4
- new net: RN?.16 (R1.2), U?.1
- new net: J?.2 (Pin_2), U?.3 (x8)
- new net: RN?.15 (R2.2), U?.1
- new net: RN?.14 (R3.2), U?.1
- new net: RN?.13 (R4.2), U?.1
- new net: RN?.12 (R5.2), U?.1
- new net: RN?.11 (R6.2), U?.1
- new net: RN?.10 (R7.2), U?.1
- new net: RN?.9 (R8.2), U?.1
- new net GNDPWR: C9.2, J10.1 (Pin_1), J?.1 (Pin_1), J?.1 (Pin_1), J?.1 (Pin_1), J?.1 (Pin_1), J?.1 (Pin_1), J?.1 (Pin_1), J?.1 (Pin_1), J?.1 (Pin_1)
Other:
- moved on the sheet: C9, F1, J10, J9, U1

Commit message: solenoid 完成
Parts:
- removed J9: usart,i2c, Connector_JST:JST_PH_S4B-PH-K_1x04_P2.00mm_Horizontal, symbol Connector:Conn_01x04_Male
- added D1: LED, LED_SMD:LED_0603_1608Metric, symbol Device:LED
- added R1: R, Resistor_SMD:R_0603_1608Metric, symbol Device:R
- J1, J2, J3, J4, J5, J6, J7, J8: renamed from J?; footprint (none) -> Connector_JST:JST_PH_S2B-PH-K_1x02_P2.00mm_Horizontal
- RN1: renamed from RN?; footprint (none) -> Resistor_SMD:R_Array_Convex_8x0602
- gave numbers to parts that had none: 8
Connections:
- net AD0: now also RN1.8 (R8.1); no longer RN1.1 (R1.1)
- net AD1: now also RN1.7 (R7.1); no longer RN1.2 (R2.1)
- net AD2: now also RN1.6 (R6.1); no longer RN1.3 (R3.1)
- net AD3: now also RN1.5 (R5.1); no longer RN1.4 (R4.1)
- net AD4: now also RN1.4 (R4.1); no longer RN1.5 (R5.1)
- net AD5: now also RN1.3 (R3.1); no longer RN1.6 (R6.1)
- net AD6: now also RN1.2 (R2.1); no longer RN1.7 (R7.1)
- net AD7: now also RN1.1 (R1.1); no longer RN1.8 (R8.1)
- net GNDPWR: now also D1.1 (K)
- net VCC: now also R1.1
- net at U2.1: now also RN1.9 (R8.2); no longer RN1.16 (R1.2)
- net at U3.1: now also RN1.10 (R7.2); no longer RN1.15 (R2.2)
- net at U4.1: now also RN1.11 (R6.2); no longer RN1.14 (R3.2)
- net at U5.1: now also RN1.12 (R5.2); no longer RN1.13 (R4.2)
- net at U6.1: now also RN1.13 (R4.2); no longer RN1.12 (R5.2)
- net at U7.1: now also RN1.14 (R3.2); no longer RN1.11 (R6.2)
- net at U8.1: now also RN1.15 (R2.2); no longer RN1.10 (R7.2)
- net at U9.1: now also RN1.16 (R1.2); no longer RN1.9 (R8.2)
- net +3V3: no longer names the net of U1.21 (3.3V)
- net PWM0: no longer names the net of U1.16 (PB4)
- net PWM1: no longer names the net of U1.17 (PB5)
- net PWM2: no longer names the net of U1.14 (PA15)
- net PWM3: no longer names the net of U1.15 (PB3)
- net PWM4: no longer names the net of U1.10 (PB1)
- net PWM5: no longer names the net of U1.9 (PB0)
- net PWM6: no longer names the net of U1.12 (PA9)
- net PWM7: no longer names the net of U1.11 (PA8)
- net PWM8: no longer names the net of U1.13 (PA10)
- net RX,SDA: no longer names the net of U1.19 (PB7)
- net TX,SCL: no longer names the net of U1.18 (PB6)
- new net: D1.2 (A), R1.2
- no-connect marks 2 -> 14
Other:
- moved on the sheet: C9, F1, J10, U1
